Commit message: [aerial_robot_simulation][ROS2][WIP] Reimplementation of AerialRobotHwSim to use gz_ros2_control's hardware interface as base class.

File: aerial_robot_simulation/xacro/spinal.gazebo.xacro (robot description, xacro)
@@ -3,13 +3,55 @@
     xmlns:xacro="http://www.ros.org/wiki/xacro" name="spinal" >
   <xacro:macro name="gazebo_spinal" params="robot_name imu_frame:=fc mag_frame:=magnet gps_frame:=gps">
-  <ros2_control name="aerial_robot_controller_manager" type="system">
+  <ros2_control name="aerial_robot_sim_system" type="system">
     <hardware>
-      <plugin>aerial_robot_simulation::AerialRobotHwSim</plugin>
+      <plugin>gz_ros2_control/AerialRobotHwSim</plugin>
     </hardware>
+    <joint name="joint1">
+      <command_interface name="position">
+        <param name="min">-15</param>
+        <param name="max">15</param>
+      </command_interface>
+      <state_interface name="position">
+        <param name="initial_value">0.0</param>
+      </state_interface>
+      <state_interface name="velocity"/>
+      <state_interface name="effort"/>
+    </joint>
+    <joint name="joint2">
+      <command_interface name="position">
+        <param name="min">-15</param>
+        <param name="max">15</param>
+      </command_interface>
+      <state_interface name="position">
+        <param name="initial_value">0.0</param>
+      </state_interface>
+      <state_interface name="velocity"/>
+      <state_interface name="effort"/>
+    </joint>
+    <joint name="joint3">
+      <command_interface name="position">
+        <param name="min">-15</param>
+        <param name="max">15</param>
+      </command_interface>
+      <state_interface name="position">
+        <param name="initial_value">0.0</param>
+      </state_interface>
+      <state_interface name="velocity"/>
+      <state_interface name="effort"/>
+    </joint>
   </ros2_control>
   <gazebo>
-    <plugin name="aerial_robot_simulation::AerialRobotIgn" filename="libaerial_robot_ign_plugin.so">
+    <plugin filename="gz_ros2_control-system" name="gz_ros2_control::GazeboSimROS2ControlPlugin">
+      <parameters>$(find aerial_robot_simulation)/config/Gazebo.yaml</parameters>
+      <ros>
+        <namespace>hydrus</namespace>
+        <!-- <remapping>/robot_description:=/robot_description_full</remapping> -->
+      </ros>
     </plugin>
   </gazebo>
+  <!-- <gazebo> -->
+  <!--   <plugin name="aerial_robot_simulation::AerialRobotIgn" filename="libaerial_robot_ign_plugin.so"> -->
+  <!--   </plugin> -->
+  <!-- </gazebo> -->
     <!-- imu plugin -->
     <!--

Commit message: [aerial_robot_simulation][ROS2][WIP] Refactor URDF configure process.

File: aerial_robot_simulation/xacro/spinal.gazebo.xacro (robot description, xacro)
@@ -3,77 +3,12 @@
     xmlns:xacro="http://www.ros.org/wiki/xacro" name="spinal" >
   <xacro:macro name="gazebo_spinal" params="robot_name imu_frame:=fc mag_frame:=magnet gps_frame:=gps">
-  <ros2_control name="aerial_robot_sim_system" type="system">
-    <hardware>
-      <plugin>gz_ros2_control/AerialRobotHwSim</plugin>
-    </hardware>
-    <joint name="joint1">
-      <command_interface name="position">
-        <param name="min">-15</param>
-        <param name="max">15</param>
-      </command_interface>
-      <state_interface name="position">
-        <param name="initial_value">0.0</param>
-      </state_interface>
-      <state_interface name="velocity"/>
-      <state_interface name="effort"/>
-    </joint>
-    <joint name="joint2">
-      <command_interface name="position">
-        <param name="min">-15</param>
-        <param name="max">15</param>
-      </command_interface>
-      <state_interface name="position">
-        <param name="initial_value">0.0</param>
-      </state_interface>
-      <state_interface name="velocity"/>
-      <state_interface name="effort"/>
-    </joint>
-    <joint name="joint3">
-      <command_interface name="position">
-        <param name="min">-15</param>
-        <param name="max">15</param>
-      </command_interface>
-      <state_interface name="position">
-        <param name="initial_value">0.0</param>
-      </state_interface>
-      <state_interface name="velocity"/>
-      <state_interface name="effort"/>
-    </joint>
-    <sensor name="spinal_imu">
-      <state_interface name="orientation.x"/>
-      <state_interface name="orientation.y"/>
-      <state_interface name="orientation.z"/>
-      <state_interface name="orientation.w"/>
-      <state_interface name="angular_velocity.x"/>
-      <state_interface name="angular_velocity.y"/>
-      <state_interface name="angular_velocity.z"/>
-      <state_interface name="linear_acceleration.x"/>
-      <state_interface name="linear_acceleration.y"/>
-      <state_interface name="linear_acceleration.z"/>
-    </sensor>
-    <sensor name="spinal_mag">
-      <state_interface name="field_tesla.x"/>
-      <state_interface name="field_tesla.y"/>
-      <state_interface name="field_tesla.z"/>
-    </sensor>
-  </ros2_control>
   <gazebo>
     <plugin filename="gz_ros2_control-system" name="gz_ros2_control::GazeboSimROS2ControlPlugin">
       <parameters>$(find aerial_robot_simulation)/config/Gazebo.yaml</parameters>
       <ros>
-        <namespace>hydrus</namespace>
-        <!-- <remapping>/robot_description:=/robot_description_full</remapping> -->
+        <namespace>${robot_name}</namespace>
       </ros>
     </plugin>
   </gazebo>
-  <!-- <gazebo> -->
-  <!--   <plugin name="aerial_robot_simulation::AerialRobotIgn" filename="libaerial_robot_ign_plugin.so"> -->
-  <!--   </plugin> -->
-  <!-- </gazebo> -->
-    <!-- imu plugin -->
-    <!--
-        note1: please do not use hector_gazebo_ros_imu, which calculates the acceleration in the parent link of the imu frame (e.g. fc -> link2)
-        note2: please do not trust the acceleration value from the multilinked model. Since the acceleration is calculated from the differential of veloctity (see https://bitbucket.org/osrf/gazebo/src/cde54284e90b59a9af9fade096946c0cd4a91c44/gazebo/sensors/ImuSensor.cc#lines-366:367). The internal force from joint create a very unstable acceleration to the link. Anyway, you can test the sensor fusio for general multirotor and transformable robot with only hovering motion.
-    -->
     <gazebo reference="${imu_frame}">
       <sensor name="spinal_imu" type="imu">

File: robots/hydrus/robots/quad/default_mode_201907/robot.urdf.xacro (robot description, xacro)
@@ -101,3 +101,29 @@
   </xacro:extra_module>
   <!-- end: gps -->
+  <ros2_control name="aerial_robot_sim_system" type="system">
+    <hardware>
+      <plugin>gz_ros2_control/AerialRobotHwSim</plugin>
+    </hardware>
+    <xacro:joint_actuation self="1"/>
+    <xacro:joint_actuation self="2"/>
+    <xacro:joint_actuation self="3"/>
+    <xacro:joint_actuation self="4"/>
+    <sensor name="spinal_imu">
+      <state_interface name="orientation.x"/>
+      <state_interface name="orientation.y"/>
+      <state_interface name="orientation.z"/>
+      <state_interface name="orientation.w"/>
+      <state_interface name="angular_velocity.x"/>
+      <state_interface name="angular_velocity.y"/>
+      <state_interface name="angular_velocity.z"/>
+      <state_interface name="linear_acceleration.x"/>
+      <state_interface name="linear_acceleration.y"/>
+      <state_interface name="linear_acceleration.z"/>
+    </sensor>
+    <sensor name="spinal_mag">
+      <state_interface name="field_tesla.x"/>
+      <state_interface name="field_tesla.y"/>
+      <state_interface name="field_tesla.z"/>
+    </sensor>
+  </ros2_control>
 </robot>

File: robots/hydrus/urdf/link.urdf.xacro (robot description, xacro)
@@ -320,32 +320,18 @@
       </joint>
     </xacro:if>
-    <!-- hardware interface -->
-    <xacro:unless value="${self == links}">
-      <transmission name="joint_tran${self}">
-        <type>transmission_interface/SimpleTransmission</type>
-        <joint name="joint${self}">
-          <!-- TODO: effort is torque, maybe position is enough -->
-          <hardwareInterface>hardware_interface/EffortJointInterface</hardwareInterface>
-        </joint>
-        <actuator name="servo{self}">
-          <!-- TODO: effort is torque, maybe position is enough -->
-          <hardwareInterface>hardware_interface/EffortJointInterface</hardwareInterface>
-          <mechanicalReduction>1</mechanicalReduction>
-        </actuator>
-      </transmission>
-    </xacro:unless>
-    <transmission name="rotor_tran${self}">
-      <type>transmission_interface/SimpleTransmission</type>
-      <joint name="rotor${self}">
-        <!-- TODO: effort is torque, maybe position is enough -->
-        <hardwareInterface>RotorInterface</hardwareInterface>
-      </joint>
-      <actuator name="rotor${self}">
-        <!-- TODO: effort is torque, maybe position is enough -->
-        <hardwareInterface>RotorInterface</hardwareInterface>
-        <mechanicalReduction>1</mechanicalReduction>
-      </actuator>
-    </transmission>
-    <xacro:friction self ="${self}"/>
+  </xacro:macro>
+  <!-- ros2_control hardware interface -->
+  <xacro:macro name="joint_actuation" params="self max:=15 min:=-15 init:=0.0">
+    <joint name="joint${self}">
+      <command_interface name="position">
+        <param name="min">"${min}"</param>
+        <param name="max">"${max}"</param>
+      </command_interface>
+      <state_interface name="position">
+        <param name="initial_value">"${init}"</param>
+      </state_interface>
+      <state_interface name="velocity"/>
+      <state_interface name="effort"/>
+    </joint>
   </xacro:macro>
 </robot>
