Commit message: [Hydrus][ROS2][WIP] Debug in joint transmission macro.

File: robots/hydrus/urdf/link.urdf.xacro (robot description, xacro)
@@ -322,12 +322,12 @@
   </xacro:macro>
   <!-- ros2_control hardware interface -->
-  <xacro:macro name="joint_actuation" params="self max:=15 min:=-15 init:=0.0">
+  <xacro:macro name="joint_actuation" params="self max_pos:=${pi/2} min_pos:=${-pi/2} init_pos:=${0.0}">
     <joint name="joint${self}">
       <command_interface name="position">
-        <param name="min">"${min}"</param>
-        <param name="max">"${max}"</param>
+        <param name="min">${max_pos}</param>
+        <param name="max">${min_pos}</param>
       </command_interface>
       <state_interface name="position">
-        <param name="initial_value">"${init}"</param>
+        <param name="initial_value">${init_pos}</param>
       </state_interface>
       <state_interface name="velocity"/>
