Commit message: [mini_quadrotor][ROS2][WIP]Workaround enabling simulation of miniquadrotor.

File: robots/mini_quadrotor/urdf/robot.gazebo.xacro (robot description, xacro)
@@ -2,7 +2,40 @@
 <robot
     xmlns:xacro="http://www.ros.org/wiki/xacro" name="mini_quadrotor" >
-  <xacro:arg name="robot_name" default="quadrotor" />
+  <xacro:arg name="robot_name" default="mini_quadrotor" />
   <!-- robot urdf -->
   <xacro:include filename="$(find mini_quadrotor)/urdf/robot.urdf.xacro" />
+  <ros2_control name="aerial_robot_sim_system" type="system">
+    <hardware>
+      <plugin>gz_ros2_control/AerialRobotHwSim</plugin>
+    </hardware>
+    <joint name="dummy_joint">
+      <command_interface name="position">
+        <param name="min">${pi/2}</param>
+        <param name="max">${-pi/2}</param>
+      </command_interface>
+      <state_interface name="position">
+        <param name="initial_value">${0}</param>
+      </state_interface>
+      <state_interface name="velocity"/>
+      <state_interface name="effort"/>
+    </joint>
+    <sensor name="spinal_imu">
+      <state_interface name="orientation.x"/>
+      <state_interface name="orientation.y"/>
+      <state_interface name="orientation.z"/>
+      <state_interface name="orientation.w"/>
+      <state_interface name="angular_velocity.x"/>
+      <state_interface name="angular_velocity.y"/>
+      <state_interface name="angular_velocity.z"/>
+      <state_interface name="linear_acceleration.x"/>
+      <state_interface name="linear_acceleration.y"/>
+      <state_interface name="linear_acceleration.z"/>
+    </sensor>
+    <sensor name="spinal_mag">
+      <state_interface name="field_tesla.x"/>
+      <state_interface name="field_tesla.y"/>
+      <state_interface name="field_tesla.z"/>
+    </sensor>
+  </ros2_control>
   <!-- gazebo plugin for default controller and sensors -->
   <xacro:include filename="$(find aerial_robot_simulation)/xacro/spinal.gazebo.xacro" />

File: robots/mini_quadrotor/urdf/robot.urdf.xacro (robot description, xacro)
@@ -93,4 +93,22 @@
     <axis xyz="0 0 1"/>
   </joint>
+  <!-- dummy link for gz_ros2_control -->
+  <link name="dummy_link">
+    <inertial>
+      <origin xyz="0 0 0" rpy="0 0 0"/>
+      <mass value="0.00001"/>
+      <inertia
+          ixx="0.000001" ixy="0.0" ixz="0.0"
+          iyy="0.000001" iyz="0.0"
+          izz="0.000002"/>
+    </inertial>
+  </link>
+  <joint name="dummy_joint" type="revolute">
+    <limit effort="10.0" lower="${-pi/2}" upper="${pi/2}" velocity="0.5"/>
+    <parent link="main_body"/>
+    <child link="dummy_link"/>
+    <origin rpy="0 0 0" xyz="0 0 0"/>
+    <axis xyz="0 0 1"/>
+  </joint>
   <!-- main_body -->
   <link name="main_body">
